File: boost/boost.kicad_sch (KiCad schematic)
At the start: 1 part, among them U1 XL6019E1

Commit message: update
Parts:
- added C1: 220uF/60V, symbol Device:C_Polarized
- added C2: 1uF, symbol Device:C
- added D1: MBRD1045, Package_TO_SOT_SMD:TO-252-2, symbol Device:D_Schottky
- added F1: 5A, symbol Device:Fuse
- added J1: Screw_Terminal_01x02, TerminalBlock_Phoenix:TerminalBlock_Phoenix_MKDS-1,5-2-5.08_1x02_P5.08mm_Horizontal, symbol Connector:Screw_Terminal_01x02
- added L1: 47uH/6A, symbol Device:L
Connections:
- net GND: now also C1.2, C2.2, J1.1 (Pin_1)
- net VCC: now also C1.1, C2.1, F1.2, L1.1
- net at U1.3 (SW): now also U1.6 (SW), D1.2 (A), L1.2
- new net: F1.1, J1.2 (Pin_2)
- no-connect marks 0 -> 1
Other:
- moved on the sheet: U1

Commit message: update
Parts:
- added C3: 1uF, symbol Device:C
- added C4: 220uF/60V, symbol Device:C_Polarized
- added J2: Screw_Terminal_01x02, TerminalBlock_Phoenix:TerminalBlock_Phoenix_MKDS-1,5-2-5.08_1x02_P5.08mm_Horizontal, symbol Connector:Screw_Terminal_01x02
- added R1: 16k, symbol Device:R
- added R2: 3k, symbol Device:R
- added R3: 125k, symbol Device:R_Variable
Connections:
- net GND: now also C3.2, C4.2, J2.2 (Pin_2), R2.2
- net at D1.1 (K): now also C3.1, C4.1, J2.1 (Pin_1), R1.1
- net at U1.5 (FB): now also R2.1, R3.2
- new net: R1.2, R3.1

Commit message: update
Parts:
- C1, C4: footprint (none) -> Capacitor_SMD:CP_Elec_10x10.5
- C2: footprint (none) -> Capacitor_SMD:C_1206_3216Metric
- D1: LCSC (none) -> C5137764
- F1: footprint (none) -> Fuse:Fuse_1206_3216Metric; LCSC (none) -> C553937
- L1: footprint (none) -> Capacitor_THT:C_Rect_L26.5mm_W11.5mm_P22.50mm_MKS4; LCSC (none) -> C18213939
- R1: value 16k -> 41k
- R2: footprint (none) -> Resistor_SMD:R_1206_3216Metric
- R3: value 125k -> 100k; footprint (none) -> Potentiometer_THT:Potentiometer_Bourns_3266Y_Vertical
Changed lines of the file:
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@@
 		)
 	)
-	(text_box "5V-40V to 8-60V 5A DC-DC"
+	(text_box "5V-40V to 18-60V 5A DC-DC"
 		(exclude_from_sim no)
 		(at 67.31 19.05 0)
@@
 			)
 		)
+		(property "LCSC" "C5137764"
+			(at 119.38 36.83 0)
+			(effects
+				(font
+					(size 1.27 1.27)
+				)
+				(hide yes)
+			)
+		)
 		(pin "2"
 		)
@@
 			)
 		)
-		(property "Value" "16k"
+		(property "Value" "41k"
 			(at 147.32 53.3399 0)
 			(effects
@@
 			)
 		)
-		(property "Footprint" ""
+		(property "Footprint" "Capacitor_SMD:C_1206_3216Metric"
 			(at 91.1352 91.44 0)
 			(effects
@@
 			)
 		)
-		(property "Value" "125k"
+		(property "Value" "100k"
 			(at 148.59 63.4999 0)
 			(effects
@@
 			)
 		)
-		(property "Footprint" ""
+		(property "Footprint" "Potentiometer_THT:Potentiometer_Bourns_3266Y_Vertical"
 			(at 143.002 62.23 90)
 			(effects
@@
 			)
 		)
-		(property "Footprint" ""
+		(property "Footprint" "Fuse:Fuse_1206_3216Metric"
 			(at 55.88 72.898 90)
 			(effects
@@
 		(property "Description" "Fuse"
 			(at 55.88 71.12 0)
+			(effects
+				(font
+					(size 1.27 1.27)
+				)
+				(hide yes)
+			)
+		)
+		(property "LCSC" "C553937"
+			(at 55.88 71.12 90)
 			(effects
 				(font
@@
 			)
 		)
-		(property "Footprint" ""
+		(property "Footprint" "Capacitor_SMD:CP_Elec_10x10.5"
 			(at 176.8348 69.85 0)
 			(effects
@@
 			)
 		)
-		(property "Footprint" ""
+		(property "Footprint" "Resistor_SMD:R_1206_3216Metric"
 			(at 143.002 86.36 90)
 			(effects
@@
 			)
 		)
-		(property "Footprint" ""
+		(property "Footprint" "Capacitor_THT:C_Rect_L26.5mm_W11.5mm_P22.50mm_MKS4"
 			(at 97.79 36.83 0)
 			(effects
@@
 		(property "Description" "Inductor"
 			(at 97.79 36.83 0)
+			(effects
+				(font
+					(size 1.27 1.27)
+				)
+				(hide yes)
+			)
+		)
+		(property "LCSC" "C18213939"
+			(at 97.79 36.83 90)
 			(effects
 				(font
@@
 			)
 		)
-		(property "Footprint" ""
+		(property "Footprint" "Capacitor_SMD:CP_Elec_10x10.5"
 			(at 73.9648 91.44 0)
 			(effects

Commit message: update
Parts:
- C3: footprint (none) -> Capacitor_SMD:C_1206_3216Metric
- R1: footprint (none) -> Resistor_SMD:R_1206_3216Metric
Changed lines of the file:
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@@
 			)
 		)
-		(property "Footprint" ""
+		(property "Footprint" "Resistor_SMD:R_1206_3216Metric"
 			(at 143.002 52.07 90)
 			(effects
@@
 			)
 		)
-		(property "Footprint" ""
+		(property "Footprint" "Capacitor_SMD:C_1206_3216Metric"
 			(at 163.5252 69.85 0)
 			(effects
