File: boost/boost.kicad_pcb (KiCad board)
At the start: 2 copper layers, 13 parts, among them J1 Screw_Terminal_01x02, J2 Screw_Terminal_01x02, U1 XL6019E1

Commit message: finish
Parts:
- moved C2 11.9 mm to (99.0, 65.5)
Routing:
- net GND: track 43.3 -> 128.3 mm
- net Vout: track 23.4 -> 80.7 mm, vias 0 -> 1
- net Vin: track 63.1 -> 75.6 mm
Other:
- board outline added: 105 x 35 mm
- board text added: "GND Vin"
- board text added: "GND Vout"
Changed lines of the file:
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@@
 	(footprint "Capacitor_SMD:C_1206_3216Metric"
 		(layer "F.Cu")
-		(at 93.475 55 180)
+		(at 99.025 65.5 180)
 		(descr "Capacitor SMD 1206 (3216 Metric), square (rectangular) end terminal, IPC_7351 nominal, (Body size source: IPC-SM-782 page 76, https://www.pcb-3d.com/wordpress/wp-content/uploads/ipc-sm-782a_amendment_1_and_2.pdf), generated with kicad-footprint-generator")
 		(tags "capacitor")
@@
 		)
 	)
+	(gr_rect
+		(start 70 55)
+		(end 175 90)
+		(stroke
+			(width 0.05)
+			(type default)
+		)
+		(fill none)
+		(layer "Edge.Cuts")
+	)
+	(gr_text "GND\n\n\n\n\n\n\n\n\nVin"
+		(at 75 78 0)
+		(layer "F.SilkS")
+		(effects
+			(font
+				(size 1 1)
+				(thickness 0.1)
+			)
+			(justify left bottom)
+		)
+	)
+	(gr_text "GND\n\n\n\n\n\n\n\n\nVout"
+		(at 166.5 77.5 0)
+		(layer "F.SilkS")
+		(effects
+			(font
+				(size 1 1)
+				(thickness 0.1)
+			)
+			(justify left bottom)
+		)
+	)
 	(segment
 		(start 160.05 78.5)
@@
 	)
 	(segment
+		(start 136.67 63.77)
+		(end 143.5 63.77)
+		(width 1.4)
+		(layer "F.Cu")
+		(net 1)
+	)
+	(segment
+		(start 136.28 56.55)
+		(end 143.5 63.77)
+		(width 1.4)
+		(layer "F.Cu")
+		(net 1)
+	)
+	(segment
+		(start 88.98 65.8)
+		(end 97.25 65.8)
+		(width 1.4)
+		(layer "F.Cu")
+		(net 1)
+	)
+	(segment
 		(start 160.05 70.35)
 		(end 155.5 65.8)
@@
 	)
 	(segment
+		(start 133.84 66.6)
+		(end 136.67 63.77)
+		(width 1.4)
+		(layer "F.Cu")
+		(net 1)
+	)
+	(segment
+		(start 97.25 65.8)
+		(end 97.55 65.5)
+		(width 1.4)
+		(layer "F.Cu")
+		(net 1)
+	)
+	(segment
 		(start 127.9625 64.5)
 		(end 131.74 64.5)
@@
 	)
 	(segment
+		(start 153.47 63.77)
+		(end 155.5 65.8)
+		(width 1.4)
+		(layer "F.Cu")
+		(net 1)
+	)
+	(segment
 		(start 162.98 67.42)
 		(end 160.05 70.35)
@@
 	)
 	(segment
+		(start 106.5 56.55)
+		(end 136.28 56.55)
+		(width 1.4)
+		(layer "F.Cu")
+		(net 1)
+	)
+	(segment
+		(start 97.55 65.5)
+		(end 106.5 56.55)
+		(width 1.4)
+		(layer "F.Cu")
+		(net 1)
+	)
+	(segment
 		(start 76.675 67.455)
 		(end 87.325 67.455)
@@
 	)
 	(segment
+		(start 143.5 63.77)
+		(end 153.47 63.77)
+		(width 1.4)
+		(layer "F.Cu")
+		(net 1)
+	)
+	(segment
 		(start 131.74 64.5)
 		(end 133.84 66.6)
@@
 	)
 	(segment
+		(start 104.625 76.375)
+		(end 111 82.75)
+		(width 1.4)
+		(layer "F.Cu")
+		(net 7)
+	)
+	(segment
 		(start 91.28 71.9)
 		(end 88.98 74.2)
@@
 	)
 	(segment
+		(start 102.255 74.005)
+		(end 104.625 76.375)
+		(width 1.4)
+		(layer "F.Cu")
+		(net 7)
+	)
+	(segment
 		(start 133.84 71.7)
 		(end 136.475 71.7)
@@
 	)
 	(segment
+		(start 102.255 67.255)
+		(end 102.255 74.005)
+		(width 1.4)
+		(layer "F.Cu")
+		(net 7)
+	)
+	(segment
 		(start 100.48 71.9)
 		(end 91.28 71.9)
@@
 	)
 	(segment
+		(start 100.5 65.5)
+		(end 102.255 67.255)
+		(width 1.4)
+		(layer "F.Cu")
+		(net 7)
+	)
+	(segment
 		(start 136.74 74.835)
 		(end 128.825 82.75)
@@
 	)
 	(segment
+		(start 100.48 72.23)
+		(end 104.625 76.375)
+		(width 1.4)
+		(layer "F.Cu")
+		(net 7)
+	)
+	(segment
 		(start 128.825 82.75)
 		(end 111 82.75)
@@
 	)
 	(segment
-		(start 100.48 72.23)
-		(end 111 82.75)
-		(width 1.4)
-		(layer "F.Cu")
-		(net 7)
+		(start 119.575 65.895)
+		(end 119.575 63.575)
+		(width 1.4)
+		(layer "F.Cu")
+		(net 8)
 	)
 	(segment
@@
 	)
 	(segment
+		(start 119.575 63.575)
+		(end 118.5 62.5)
+		(width 1.4)
+		(layer "F.Cu")
+		(net 8)
+	)
+	(segment
 		(start 163 78.5)
 		(end 161.2 80.3)
@@
 		(net 8)
 	)
+	(via
+		(at 118.5 62.5)
+		(size 1.4)
+		(drill 0.8)
+		(layers "F.Cu" "B.Cu")
+		(net 8)
+	)
+	(segment
+		(start 128.5 72.5)
+		(end 118.5 62.5)
+		(width 1.4)
+		(layer "B.Cu")
+		(net 8)
+	)
+	(segment
+		(start 167.805 72.5)
+		(end 128.5 72.5)
+		(width 1.4)
+		(layer "B.Cu")
+		(net 8)
+	)

Commit message: fix
Routing:
- net GND: track 128.3 -> 133.0 mm, vias 0 -> 12
- added copper zone on B.Cu, net GND
- added copper zone on F.Cu, net GND
