File: buck/buck.kicad_sch (KiCad schematic)
At the start: 2 parts, among them U1 LM2596S-12

Commit message: update
Parts:
- added C1: 680uF/50V, symbol Device:C_Polarized
- added C2: 260uF/35V, symbol Device:C_Polarized
- added C3: C, symbol Device:C
- added D1: ss34, symbol Device:D_Schottky
- added J1, J2: Screw_Terminal_01x02, TerminalBlock_Phoenix:TerminalBlock_Phoenix_MKDS-1,5-2-5.08_1x02_P5.08mm_Horizontal, symbol Connector:Screw_Terminal_01x02
- added R1: 1k, symbol Device:R
- added R2: 3k, symbol Device:R
- added R3: 10k, symbol Device:R_Variable
- L1: value L -> 470
Connections:
- net VCC: now reaches U1.1 (VIN)
- net VCC: now also C1.1, J2.2 (Pin_2)
- net at U1.2 (OUT): now also L1.1, D1.1 (K)
- net GND: now reaches U1.3 (GND)
- net GND: now also U1.5 (~{ON}/OFF), C1.2, C2.2, D1.2 (A), J1.2 (Pin_2), J2.1 (Pin_1), R1.1
- net at U1.4 (FB): now also C3.1, R1.2, R3.2
- net Vout: now reaches L1.2
- net Vout: now also C2.1, C3.2, J1.1 (Pin_1), R2.2
- new net: R2.1, R3.1
Other:
- moved on the sheet: L1, U1

Commit message: update
Parts:
- C3: value C -> 2.2uF/50V
Changed lines of the file:
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@@
 			)
 		)
-		(property "Value" "C"
+		(property "Value" "2.2uF/50V"
 			(at 115.57 20.32 90)
 			(effects

Commit message: update
Parts:
- C1: footprint (none) -> Capacitor_SMD:CP_Elec_10x12.5
- C2: value 260uF/35V -> 220uF/35V; footprint (none) -> Capacitor_SMD:C_Elec_8x10.2
- C3: footprint (none) -> Capacitor_SMD:C_0201_0603Metric
- D1: footprint (none) -> Diode_SMD:D_SMA
- R1, R2: footprint (none) -> Resistor_SMD:R_1206_3216Metric
- R3: footprint (none) -> Potentiometer_THT:Potentiometer_Bourns_3296W_Vertical
Changed lines of the file:
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@@
 			)
 		)
-		(property "Footprint" ""
+		(property "Footprint" "Capacitor_SMD:C_0201_0603Metric"
 			(at 119.38 24.4348 0)
 			(effects
@@
 			)
 		)
-		(property "Footprint" ""
+		(property "Footprint" "Capacitor_SMD:CP_Elec_10x12.5"
 			(at 78.4352 57.15 0)
 			(effects
@@
 			)
 		)
-		(property "Footprint" ""
+		(property "Footprint" "Diode_SMD:D_SMA"
 			(at 125.73 55.88 0)
 			(effects
@@
 			)
 		)
-		(property "Footprint" ""
+		(property "Footprint" "Resistor_SMD:R_1206_3216Metric"
 			(at 120.65 37.338 90)
 			(effects
@@
 			)
 		)
-		(property "Footprint" ""
+		(property "Footprint" "Potentiometer_THT:Potentiometer_Bourns_3296W_Vertical"
 			(at 111.76 33.782 90)
 			(effects
@@
 			)
 		)
-		(property "Footprint" ""
+		(property "Footprint" "Resistor_SMD:R_1206_3216Metric"
 			(at 97.79 37.338 90)
 			(effects
@@
 			)
 		)
-		(property "Value" "260uF/35V"
+		(property "Value" "220uF/35V"
 			(at 143.51 56.2609 0)
 			(effects
@@
 			)
 		)
-		(property "Footprint" ""
+		(property "Footprint" "Capacitor_SMD:C_Elec_8x10.2"
 			(at 140.6652 59.69 0)
 			(effects

Commit message: update
Parts:
- L1: footprint (none) -> Inductor_SMD:L_SXN_SMDRI127
Other:
- moved on the sheet: L1
Changed lines of the file:
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@@
+	(wire
+		(pts
+			(xy 138.43 52.07) (xy 139.7 52.07)
+		)
+		(stroke
+			(width 0)
+			(type default)
+		)
+	)
 	(wire
 		(pts
@@
 	(wire
 		(pts
-			(xy 125.73 52.07) (xy 132.08 52.07)
+			(xy 125.73 52.07) (xy 130.81 52.07)
 		)
 		(stroke
@@
 	(symbol
 		(lib_id "Device:L")
-		(at 135.89 52.07 90)
+		(at 134.62 52.07 90)
 		(unit 1)
 		(exclude_from_sim no)
@@
 		(fields_autoplaced yes)
 		(property "Reference" "L1"
-			(at 135.89 46.99 90)
+			(at 134.62 46.99 90)
 			(effects
 				(font
@@
 		)
 		(property "Value" "470"
-			(at 135.89 49.53 90)
-			(effects
-				(font
-					(size 1.27 1.27)
-				)
-			)
-		)
-		(property "Footprint" ""
-			(at 135.89 52.07 0)
+			(at 134.62 49.53 90)
+			(effects
+				(font
+					(size 1.27 1.27)
+				)
+			)
+		)
+		(property "Footprint" "Inductor_SMD:L_SXN_SMDRI127"
+			(at 134.62 52.07 0)
 			(effects
 				(font
@@
 		)
 		(property "Datasheet" "~"
-			(at 135.89 52.07 0)
+			(at 134.62 52.07 0)
 			(effects
 				(font
@@
 		)
 		(property "Description" "Inductor"
-			(at 135.89 52.07 0)
-			(effects
-				(font
+			(at 134.62 52.07 0)
+			(effects
+				(font

Commit message: update
Parts:
- removed R2: 3k, Resistor_SMD:R_1206_3216Metric, symbol Device:R
Connections:
- net Vout: now also R3.1
Changed lines of the file:
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@@
 	(wire
 		(pts
-			(xy 116.84 35.56) (xy 115.57 35.56)
+			(xy 115.57 35.56) (xy 127 35.56)
 		)
 		(stroke
@@
 		(pts
 			(xy 101.6 35.56) (xy 106.68 35.56)
-		)
-		(stroke
-			(width 0)
-			(type default)
-		)
-	)
-	(wire
-		(pts
-			(xy 127 35.56) (xy 124.46 35.56)
 		)
 		(stroke
@@
 					(unit 1)
 				)
-			)
-		)
-	)
-	(symbol
-		(lib_id "Device:R")
-		(at 120.65 35.56 90)
-		(unit 1)
-		(exclude_from_sim no)
-		(in_bom yes)
-		(on_board yes)
-		(dnp no)
-		(fields_autoplaced yes)
-		(property "Reference" "R2"
-			(at 120.65 29.21 90)
-			(effects
-				(font
-					(size 1.27 1.27)
-				)
-			)
-		)
-		(property "Value" "3k"
-			(at 120.65 31.75 90)
-			(effects
-				(font
-					(size 1.27 1.27)
-				)
-			)
-		)
-		(property "Footprint" "Resistor_SMD:R_1206_3216Metric"
-			(at 120.65 37.338 90)
-			(effects
-				(font
-					(size 1.27 1.27)
-				)
-				(hide yes)
-			)
-		)
-		(property "Datasheet" "~"
-			(at 120.65 35.56 0)
-			(effects
-				(font
-					(size 1.27 1.27)
-				)
-				(hide yes)
-			)
-		)
-		(property "Description" "Resistor"
-			(at 120.65 35.56 0)
-			(effects
-				(font
-					(size 1.27 1.27)
-				)
-				(hide yes)
-			)
-		)
-		(pin "1"
-		)
-		(pin "2"
-		)
-		(instances
-			(project "buck"
-				(path "/534ccee1-9696-4739-b4aa-2cab67d4d410"
-					(reference "R2")
-					(unit 1)
-				)
