File: buck/buck.kicad_pcb (KiCad board)
At the start: 2 copper layers, 11 parts, among them J1 Screw_Terminal_01x02, J2 Screw_Terminal_01x02, U1 LM2596S-12

Commit message: update
Parts:
- moved D1 71.3 mm to (77.5, 97.0)
- moved C3 57.1 mm to (96.3, 84.0)
Routing:
- net Net-(D1-K): track 0.00 -> 6.25 mm
- net GND: track 0.00 -> 5.71 mm
Changed lines of the file:
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@@
 	(footprint "Diode_SMD:D_SMA"
 		(layer "F.Cu")
-		(at 148.8025 95.29)
+		(at 77.5 97)
 		(descr "Diode SMA (DO-214AC)")
 		(tags "Diode SMA (DO-214AC)")
@@
 	(footprint "Capacitor_SMD:C_0201_0603Metric"
 		(layer "F.Cu")
-		(at 151.5675 98.44)
+		(at 96.345 84)
 		(descr "Capacitor SMD 0201 (0603 Metric), square (rectangular) end terminal, IPC_7351 nominal, (Body size source: https://www.vishay.com/docs/20052/crcw0201e3.pdf), generated with kicad-footprint-generator")
 		(tags "capacitor")
@@
 		)
 	)
+	(segment
+		(start 79 96.5)
+		(end 79.5 97)
+		(width 1.4)
+		(layer "F.Cu")
+		(net 2)
+	)
+	(segment
+		(start 79 91.5)
+		(end 79 96.5)
+		(width 1.4)
+		(layer "F.Cu")
+		(net 2)
+	)
+	(segment
+		(start 77.3 91.5)
+		(end 77.3 95.2)
+		(width 1.4)
+		(layer "F.Cu")
+		(net 5)
+	)
+	(segment
+		(start 77.3 95.2)
+		(end 75.5 97)
+		(width 1.4)
+		(layer "F.Cu")
+		(net 5)
+	)
 )

Commit message: update
Parts:
- removed R2: 3k, Resistor_SMD:R_1206_3216Metric
- moved J2 83.4 mm to (55.0, 85.0), turned to -90 degrees
- moved C2 26.7 mm to (105.0, 87.5), turned to 90 degrees
- moved J1 18.8 mm to (117.5, 90.0), turned to 90 degrees
- moved C3 2.50 mm to (93.8, 84.0)
Connections:
- R3 pad 1: Net-(R2-Pad1) -> Vout
Routing:
- net Vout: track 0.00 -> 46.7 mm
- net Net-(U1-FB): track 0.00 -> 40.2 mm
- net Net-(D1-K): track 6.25 -> 28.1 mm
- net Vin: track 0.00 -> 21.2 mm
- net GND: track 5.71 -> 2.15 mm, vias 0 -> 59
- added copper zone on B.Cu, net GND
- added copper zone on F.Cu, net GND
Other:
- board outline added: 72.5 x 27.5 mm

Commit message: fix
Other:
- board text added: "GND Vin"
- board text added: "GND Vout"
Changed lines of the file:
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@@
 		(tags "Potentiometer vertical Bourns 3296W")
 		(property "Reference" "R3"
-			(at -2.54 -3.66 360)
+			(at -2.54 -3.66 0)
 			(layer "F.SilkS")
 			(effects
@@
 		)
 		(property "Value" "10k"
-			(at -2.54 3.67 360)
+			(at -2.54 3.67 0)
 			(layer "F.Fab")
 			(effects
@@
 		)
 		(fp_text user "${REFERENCE}"
-			(at -3.175 0.005 360)
+			(at -3.175 0.005 0)
 			(layer "F.Fab")
 			(effects
@@
 		(layer "Edge.Cuts")
 	)
+	(gr_text "GND\n\n\n\n\n\n\n\n\nVout"
+		(at 116 95 0)
+		(layer "F.SilkS")
+		(effects
+			(font
+				(size 1 1)
+				(thickness 0.1)
+			)
+			(justify left bottom)
+		)
+	)
+	(gr_text "GND\n\n\n\n\n\n\n\n\nVin"
+		(at -38 96 0)
+		(layer "F.SilkS")
+		(effects
+			(font
+				(size 1 1)
+				(thickness 0.1)
+			)
+			(justify left bottom)
+		)
+	)
+	(gr_text "GND\n\n\n\n\n\n\n\n\nVin"
+		(at 54 95.5 0)
+		(layer "F.SilkS")
+		(effects
+			(font
+				(size 1 1)
+				(thickness 0.1)
+			)
+			(justify left bottom)
+		)
+	)
 	(segment
 		(start 67 90.7)
@@
 			)
 		)
-	)
-	(zone
-		(net 0)
-		(net_name "")
-		(layer "B.Cu")
-		(hatch edge 0.5)
-		(connect_pads
-			(clearance 0)
-		)
-		(min_thickness 0.25)
-		(filled_areas_thickness no)
-		(keepout
-			(tracks not_allowed)
-			(vias not_allowed)
-			(pads not_allowed)
-			(copperpour allowed)
-			(footprints allowed)
-		)
-		(fill
-			(thermal_gap 0.5)
-			(thermal_bridge_width 0.5)
-		)
-		(polygon
-			(pts
-				(xy 120 87.5) (xy 120 92.5) (xy 115 92.5) (xy 115 87.5)
-			)
-		)
-	)
-	(zone
-		(net 0)
-		(net_name "")
-		(layer "B.Cu")
-		(hatch edge 0.5)
-		(connect_pads
-			(clearance 0)
-		)
-		(min_thickness 0.25)
-		(filled_areas_thickness no)
-		(keepout
-			(tracks not_allowed)
-			(vias not_allowed)
-			(pads not_allowed)
-			(copperpour allowed)
-			(footprints allowed)
-		)
-		(fill
-			(thermal_gap 0.5)
-			(thermal_bridge_width 0.5)
-		)
-		(polygon
-			(pts
-				(xy 52.5 87.5) (xy 57.5 87.5) (xy 57.5 92.5) (xy 52.5 92.5)
-			)
-		)
